Commit message: Update xacro for new joint configuration.

File: steer_drive_controller/test/common/urdf/steerbot.xacro (robot description, xacro)
@@ -52,19 +52,27 @@
     <parent link="base_footprint"/>
   </joint>
+  <!-- joints for steer_drive_controller -->
+  <front_steer name="front" parent="base" radius="${wheel_radius}" thickness="${thickness}"
+      length="${length}" width="${width}" axel_offset="${axel_offset}" steer_height="${wheel_radius+steer_offset}">
+    <origin xyz="${length/2-axel_offset} 0 0" rpy="${-90 * deg_to_rad} 0 0"/>
+  </front_steer>
+  <rear_wheel name="rear" parent="base" radius="${wheel_radius}" thickness="${thickness}">
+    <origin xyz="${-length/2+axel_offset} 0 0" rpy="${-90 * deg_to_rad} 0 0"/>
+  </rear_wheel>
   <!-- Wheels -->
-  <front_wheel name="front_right" parent="base" radius="${wheel_radius}" thickness="${thickness}"
+  <front_wheel_lr name="front_right" parent="base" radius="${wheel_radius}" thickness="${thickness}"
       length="${length}" width="${width}" axel_offset="${axel_offset}" right_left="1" steer_height="${wheel_radius+steer_offset}">
     <origin xyz="${length/2-axel_offset} ${width/2+axel_offset} 0" rpy="${-90 * deg_to_rad} 0 0"/>
-  </front_wheel>
-  <front_wheel name="front_left" parent="base" radius="${wheel_radius}" thickness="${thickness}"
+  </front_wheel_lr>
+  <front_wheel_lr name="front_left" parent="base" radius="${wheel_radius}" thickness="${thickness}"
       length="${length}" width="${width}" axel_offset="${axel_offset}" right_left="-1" steer_height="${wheel_radius+steer_offset}">
     <origin xyz="${length/2-axel_offset} ${-width/2-axel_offset} 0" rpy="${-90 * deg_to_rad} 0 0"/>
-  </front_wheel>
-  <rear_wheel name="rear_right" parent="base" radius="${wheel_radius}" thickness="${thickness}">
+  </front_wheel_lr>
+  <rear_wheel_lr name="rear_right" parent="base" radius="${wheel_radius}" thickness="${thickness}">
     <origin xyz="${-length/2+axel_offset} ${width/2+axel_offset} 0" rpy="${-90 * deg_to_rad} 0 0"/>
-  </rear_wheel>
-  <rear_wheel name="rear_left" parent="base" radius="${wheel_radius}" thickness="${thickness}">
+  </rear_wheel_lr>
+  <rear_wheel_lr name="rear_left" parent="base" radius="${wheel_radius}" thickness="${thickness}">
     <origin xyz="${-length/2+axel_offset} ${-width/2-axel_offset} 0" rpy="${-90 * deg_to_rad} 0 0"/>
-  </rear_wheel>
+  </rear_wheel_lr>
   <!-- Colour -->
   <gazebo reference="base_link">

File: steer_drive_controller/test/common/urdf/wheel.xacro (robot description, xacro)
@@ -5,5 +5,38 @@
   <xacro:property name="steer_effort"   value="10.0"/>
   <xacro:property name="steer_velocity" value="5.0"/>
-  <macro name="front_wheel" params="name parent radius thickness length width axel_offset right_left steer_height *origin">
+  <macro name="front_steer" params="name parent radius thickness length width axel_offset steer_height *origin">
+    <link name="${name}_steer_link">
+      <inertial>
+        <origin xyz="0 0 0" rpy="0 0 0"/>
+        <mass value="1"/>
+        <inertia ixx="0.2" ixy="0" ixz="0" iyy="0.2" iyz="0" izz="0.2"/>
+      </inertial>
+      <visual>
+        <origin xyz="0 0 0" rpy="0 0 0"/>
+        <geometry>
+          <cylinder radius="${steer_radius}" length="${steer_thickness}"/>
+        </geometry>
+      </visual>
+      <collision>
+        <origin xyz="0 0 0" rpy="0 0 0"/>
+        <geometry>
+          <cylinder radius="${steer_radius}" length="${steer_thickness}"/>
+        </geometry>
+      </collision>
+    </link>
+    <joint name="${name}_steer_joint" type="revolute">
+      <parent link="${parent}_link"/>
+      <child link="${name}_steer_link"/>
+      <origin xyz="${length/2-axel_offset} 0 ${steer_height}" rpy="0 0 0"/>
+      <axis xyz="0 0 1"/>
+      <limit effort="${steer_effort}"
+             lower="${-180.0 * deg_to_rad}" upper="${180.0 * deg_to_rad}"
+             velocity="${steer_velocity}"/>
+     </joint>
+    <gazebo reference="${name}_steer_link">
+      <material>Gazebo/Yellow</material>
+    </gazebo>
+  </macro>
+  <macro name="front_wheel_lr" params="name parent radius thickness length width axel_offset right_left steer_height *origin">
     <link name="${name}_steer_link">
       <inertial>
@@ -114,4 +147,41 @@
     </transmission>
     <gazebo reference="${name}_wheel_link">
+      <material>Gazebo/Yellow</material>
+    </gazebo>
+  </macro>
+  <macro name="rear_wheel_lr" params="name parent radius thickness *origin">
+    <link name="${name}_wheel_link">
+      <inertial>
+        <origin xyz="0 0 0" rpy="0 0 0"/>
+        <mass value="1"/>
+        <inertia ixx="0.2" ixy="0" ixz="0" iyy="0.2" iyz="0" izz="0.2"/>
+      </inertial>
+      <visual>
+        <origin xyz="0 0 0" rpy="0 0 0"/>
+        <geometry>
+          <cylinder radius="${wheel_radius}" length="${thickness}"/>
+        </geometry>
+      </visual>
+      <collision>
+        <origin xyz="0 0 0" rpy="0 0 0"/>
+        <geometry>
+          <cylinder radius="${wheel_radius}" length="${thickness}"/>
+        </geometry>
+      </collision>
+    </link>
+    <joint name="${name}_wheel_joint" type="continuous">
+      <parent link="${parent}_link"/>
+      <child link="${name}_wheel_link"/>
+      <insert_block name="origin"/>
+      <axis xyz="0 0 1"/>
+    </joint>
+    <!-- Transmission is important to link the joints and the controller -->
+    <transmission name="${name}_wheel_joint_trans" type="SimpleTransmission">
+      <actuator name="${name}_wheel_joint_motor"/>
+      <joint name="${name}_wheel_joint"/>
+      <mechanicalReduction>1</mechanicalReduction>
+      <motorTorqueConstant>1</motorTorqueConstant>
+    </transmission>
+    <gazebo reference="${name}_wheel_link">
       <material>Gazebo/Red</material>
     </gazebo>
