Commit message: Update macro to xacro:macro

File: steer_drive_controller/test/common/urdf/wheel.xacro (robot description, xacro)
@@ -5,5 +5,5 @@
   <xacro:property name="steer_effort"   value="10.0"/>
   <xacro:property name="steer_velocity" value="5.0"/>
-  <macro name="front_steer" params="name parent radius thickness length width axel_offset steer_height *origin">
+  <xacro:macro name="front_steer" params="name parent radius thickness length width axel_offset steer_height *origin">
     <link name="${name}_steer_link">
       <inertial>
@@ -37,6 +37,6 @@
       <material>Gazebo/Yellow</material>
     </gazebo>
-  </macro>
-  <macro name="front_wheel_lr" params="name parent radius thickness length width axel_offset right_left steer_height *origin">
+  </xacro:macro>
+  <xacro:macro name="front_wheel_lr" params="name parent radius thickness length width axel_offset right_left steer_height *origin">
     <link name="${name}_steer_link">
       <inertial>
@@ -112,6 +112,6 @@
       <material>Gazebo/Red</material>
     </gazebo>
-  </macro>
-  <macro name="rear_wheel" params="name parent radius thickness *origin">
+  </xacro:macro>
+  <xacro:macro name="rear_wheel" params="name parent radius thickness *origin">
     <link name="${name}_wheel_link">
       <inertial>
@@ -149,6 +149,6 @@
       <material>Gazebo/Yellow</material>
     </gazebo>
-  </macro>
-  <macro name="rear_wheel_lr" params="name parent radius thickness *origin">
+  </xacro:macro>
+  <xacro:macro name="rear_wheel_lr" params="name parent radius thickness *origin">
     <link name="${name}_wheel_link">
       <inertial>
@@ -186,4 +186,4 @@
       <material>Gazebo/Red</material>
     </gazebo>
-  </macro>
+  </xacro:macro>
 </robot>

File: steer_drive_controller/test/common/urdf/wheel_sphere.xacro (robot description, xacro)
@@ -5,5 +5,5 @@
   <xacro:property name="steer_effort"   value="10.0"/>
   <xacro:property name="steer_velocity" value="5.0"/>
-  <macro name="front_steer" params="name parent radius thickness length width axel_offset steer_height *origin">
+  <xacro:macro name="front_steer" params="name parent radius thickness length width axel_offset steer_height *origin">
     <link name="${name}_steer_link">
       <inertial>
@@ -37,6 +37,6 @@
       <material>Gazebo/Yellow</material>
     </gazebo>
-  </macro>
-  <macro name="front_wheel_lr" params="name parent radius thickness length width axel_offset right_left steer_height *origin">
+  </xacro:macro>
+  <xacro:macro name="front_wheel_lr" params="name parent radius thickness length width axel_offset right_left steer_height *origin">
     <link name="${name}_steer_link">
       <inertial>
@@ -112,6 +112,6 @@
       <material>Gazebo/Red</material>
     </gazebo>
-  </macro>
-  <macro name="rear_wheel" params="name parent radius thickness *origin">
+  </xacro:macro>
+  <xacro:macro name="rear_wheel" params="name parent radius thickness *origin">
     <link name="${name}_wheel_link">
       <inertial>
@@ -149,6 +149,6 @@
       <material>Gazebo/Yellow</material>
     </gazebo>
-  </macro>
-  <macro name="rear_wheel_lr" params="name parent radius thickness *origin">
+  </xacro:macro>
+  <xacro:macro name="rear_wheel_lr" params="name parent radius thickness *origin">
     <link name="${name}_wheel_link">
       <inertial>
@@ -186,4 +186,4 @@
       <material>Gazebo/Red</material>
     </gazebo>
-  </macro>
+  </xacro:macro>
 </robot>
